Commit message: velmwheel_gazebo: Added contact plugin which detects collisions with robot's base

File: src/velmwheel/sim/velmwheel_gazebo/velmwheel_gazebo/urdf/velmwheel.urdf.xacro (robot description, xacro)
@@ -5,5 +5,5 @@
   - @maintainer Krzysztof Pierczyk (krzysztof.pierczyk@gmail.com)
   - @date       Wednesday, 9th March 2022 7:42:42 pm
-  - @modified   Wednesday, 25th May 2022 11:44:59 pm
+  - @modified   Monday, 13th March 2023 8:08:16 am
   - @project    engineering-thesis
   - @brief      Definition of the Gazebo plugins for URDF model of the WUT Velmwheel robot
@@ -87,4 +87,10 @@
             </material>
         </visual>
+        <sensor name='base_contact_sensor' type='contact'>
+            <plugin name="contact_plugin" filename="libcontact_gazebo.so"/>
+            <contact>
+                <collision>base_link_fixed_joint_lump__base_collision</collision>
+            </contact>
+        </sensor>
     </gazebo>
     <!-- Mobile front -->

Commit message: Add contact sensor for wheels

File: src/velmwheel/sim/velmwheel_gazebo/velmwheel_gazebo/urdf/velmwheel.urdf.xacro (robot description, xacro)
@@ -50,4 +50,10 @@
 				</surface>
 			</collision>
+            <sensor name='${dir}_${side}_wheel_contact_sensor' type='contact'>
+                <plugin name="${dir}_${side}_contact_plugin" filename="libcontact_gazebo.so"/>
+                <contact>
+                    <collision>wheel_${dir}${side}_collision</collision>
+                </contact>
+            </sensor>
         </gazebo>
         <gazebo reference="wheel_${dir}${side}_rollers">
